Commit message: Add grippers

File: setup/catkin/princeton_cell/urdf/abb_on_axis.urdf (robot description, URDF)
Before this commit: robot abb_on_axis, 11 links, 10 joints
Joints:
- joint abb_joint: origin xyz=0 0 0  rpy=0 0 1.57079632679  -> xyz=0 0 0  rpy=0 0 1.5707963267948966 
- joint cart_joint: limit lower=-1.926 upper=0.675 effort=100000 velocity=2.618 -> lower=0 upper=4.0 effort=100000 velocity=2.618

File: setup/catkin/princeton_cell/urdf/abb_on_axis.xacro (robot description, xacro)
@@ -1,4 +1,4 @@
 <?xml version="1.0"?>
-<robot name="princeton_cell" xmlns:xacro="http://wiki.ros.org/xacro">
+<robot name="abb_on_axis" xmlns:xacro="http://wiki.ros.org/xacro">
   <xacro:include filename="$(find princeton_cell)/urdf/abb_on_axis_macro.xacro"/>
   <xacro:abb_on_axis prefix="" />

File: setup/catkin/princeton_cell/urdf/abb_on_axis_macro.xacro (robot description, xacro)
@@ -1,8 +1,9 @@
 <?xml version="1.0"?>
 <robot xmlns:xacro="http://wiki.ros.org/xacro">
-  <xacro:macro name="princeton_cell" params="prefix">
+  <xacro:macro name="abb_on_axis" params="prefix">
     <xacro:include filename="$(find abb_resources)/urdf/common_materials.xacro"/>
     <xacro:include filename="$(find abb_irb4600_40_255)/urdf/abb_irb4600_40_255_macro.xacro"/>
     <xacro:include filename="$(find princeton_cell)/urdf/linear_axis.xacro"/>
+    <xacro:include filename="$(find princeton_cell)/urdf/gripper.xacro" />
     <xacro:linear_axis prefix="${prefix}"/>
     <joint name="${prefix}abb_joint" type="fixed">
@@ -13,4 +14,5 @@
     </joint>
     <xacro:abb_irb4600_40_255 prefix="${prefix}"/>
+    <xacro:gripper prefix="${prefix}" connected_to="${prefix}tool0"/>
   </xacro:macro>
 </robot>

File: setup/catkin/princeton_cell/urdf/princeton_cell.urdf (robot description, URDF)
Before this commit: robot full_cell, 23 links, 22 joints
Links:
- added link A_gripper; collision mesh filename=package://princeton_cell/meshes/collision/gripper.stl; visual mesh filename=package://princeton_cell/meshes/visual/gripper.stl
- added link A_tcp
- added link B_gripper; collision mesh filename=package://princeton_cell/meshes/collision/gripper.stl; visual mesh filename=package://princeton_cell/meshes/visual/gripper.stl
- added link B_tcp
Joints:
- added joint A_gripper_joint: type fixed, parent A_tool0, child A_gripper, origin xyz=0 0 0 rpy=0 0 0
- added joint A_tcp_joint: type fixed, parent A_gripper, child A_tcp, origin xyz=0 0 0.3 rpy=0 0 0
- added joint B_gripper_joint: type fixed, parent B_tool0, child B_gripper, origin xyz=0 0 0 rpy=0 0 0
- added joint B_tcp_joint: type fixed, parent B_gripper, child B_tcp, origin xyz=0 0 0.3 rpy=0 0 0
- joint A_abb_joint: origin xyz=0 0 0  rpy=0 0 1.57079632679  -> xyz=0 0 0  rpy=0 0 1.5707963267948966 
- joint A_cart_joint: limit lower=0.0 upper=4.0 effort=100000 velocity=2.618 -> lower=0 upper=4.0 effort=100000 velocity=2.618
- joint B_abb_joint: origin xyz=0 0 0  rpy=0 0 1.57079632679  -> xyz=0 0 0  rpy=0 0 1.5707963267948966 
- joint B_cart_joint: limit lower=0.0 upper=4.0 effort=100000 velocity=2.618 -> lower=0 upper=4.0 effort=100000 velocity=2.618

File: setup/catkin/princeton_cell/urdf/princeton_cell_macro.xacro (robot description, xacro)
@@ -1,7 +1,6 @@
 <?xml version="1.0"?>
 <robot xmlns:xacro="http://wiki.ros.org/xacro">
-  <xacro:macro name="full_cell">
-    <xacro:include filename="$(find princeton_cell)/urdf/abb_on_axis.xacro"/>
-<!-- =================================================================================== -->
+  <xacro:macro name="princeton_cell">
+    <xacro:include filename="$(find princeton_cell)/urdf/abb_on_axis_macro.xacro"/>
     <link name="world" />
     <joint name="A_world_joint" type="fixed">

Commit message: Rename robots to r1 and r2 and align zero of the tracks  - the geometry of the r1 track is now flipped, the belt should be on the outer side, will fix it later

File: setup/catkin/princeton_cell/urdf/abb_on_axis.urdf (robot description, URDF)
Before this commit: robot abb_on_axis, 11 links, 10 joints
Links:
- added link gripper; collision mesh filename=package://princeton_cell/meshes/collision/gripper.stl; visual mesh filename=package://princeton_cell/meshes/visual/gripper.stl
- added link tcp
Joints:
- added joint gripper_joint: type fixed, parent tool0, child gripper, origin xyz=0 0 0 rpy=0 0 0
- added joint tcp_joint: type fixed, parent gripper, child tcp, origin xyz=0 0 0.3 rpy=0 0 0
- joint abb_joint: origin xyz=0 0 0  rpy=0 0 1.5707963267948966  -> xyz=0 0 0  rpy=0 0 0
- joint cart_joint: origin xyz=0 0 0 rpy=0 0 0  -> xyz=0 0 0 rpy=0 0 0

File: setup/catkin/princeton_cell/urdf/abb_on_axis.xacro (robot description, xacro)
@@ -2,4 +2,4 @@
 <robot name="abb_on_axis" xmlns:xacro="http://wiki.ros.org/xacro">
   <xacro:include filename="$(find princeton_cell)/urdf/abb_on_axis_macro.xacro"/>
-  <xacro:abb_on_axis prefix="" />
+  <xacro:abb_on_axis prefix="" cart_yaw="0" />
 </robot>

File: setup/catkin/princeton_cell/urdf/abb_on_axis_macro.xacro (robot description, xacro)
@@ -1,5 +1,5 @@
 <?xml version="1.0"?>
 <robot xmlns:xacro="http://wiki.ros.org/xacro">
-  <xacro:macro name="abb_on_axis" params="prefix">
+  <xacro:macro name="abb_on_axis" params="prefix cart_yaw">
     <xacro:include filename="$(find abb_resources)/urdf/common_materials.xacro"/>
     <xacro:include filename="$(find abb_irb4600_40_255)/urdf/abb_irb4600_40_255_macro.xacro"/>
@@ -10,5 +10,5 @@
       <parent link="${prefix}cart"/>
       <child  link="${prefix}base_link"/>
-      <origin xyz="0 0 0 " rpy="0 0 ${pi/2} "/>
+      <origin xyz="0 0 0 " rpy="0 0 ${cart_yaw}"/>
       <dynamics damping="0.2" friction="0" />
     </joint>

File: setup/catkin/princeton_cell/urdf/princeton_cell.urdf (robot description, URDF)
Before this commit: robot princeton_cell, 27 links, 26 joints
Links:
- removed link A_axis
- removed link A_base
- removed link A_base_link
- removed link A_cart
- removed link A_gripper
- removed link A_link_1
- removed link A_link_2
- removed link A_link_3
- removed link A_link_4
- removed link A_link_5
- removed link A_link_6
- removed link A_tcp
- removed link A_tool0
- removed link B_axis
- removed link B_base
- removed link B_base_link
- removed link B_cart
- removed link B_gripper
- removed link B_link_1
- removed link B_link_2
- removed link B_link_3
- removed link B_link_4
- removed link B_link_5
- removed link B_link_6
- removed link B_tcp
- removed link B_tool0
- added link r1_axis, mass 120; collision mesh filename=package://princeton_cell/meshes/collision/axis.stl; visual mesh filename=package://princeton_cell/meshes/visual/axis.stl
- added link r1_base
- added link r1_base_link, mass 120.00000; collision mesh filename=package://abb_irb4600_40_255/meshes/collision/base_link.stl; visual mesh filename=package://abb_irb4600_40_255/meshes/visual/base_link.stl
- added link r1_cart, mass 120.00000; collision mesh filename=package://princeton_cell/meshes/collision/cart.stl; visual mesh filename=package://princeton_cell/meshes/visual/cart.stl
- added link r1_gripper; collision mesh filename=package://princeton_cell/meshes/collision/gripper.stl; visual mesh filename=package://princeton_cell/meshes/visual/gripper.stl
- added link r1_link_1, mass 120.00000; collision mesh filename=package://abb_irb4600_40_255/meshes/collision/link_1.stl; visual mesh filename=package://abb_irb4600_40_255/meshes/visual/link_1.stl
- added link r1_link_2, mass 120.00000; collision mesh filename=package://abb_irb4600_40_255/meshes/collision/link_2.stl; visual mesh filename=package://abb_irb4600_40_255/meshes/visual/link_2.stl
- added link r1_link_3, mass 120.00000; collision mesh filename=package://abb_irb4600_40_255/meshes/collision/link_3.stl; visual mesh filename=package://abb_irb4600_40_255/meshes/visual/link_3.stl
- added link r1_link_4, mass 40.00000; collision mesh filename=package://abb_irb4600_40_255/meshes/collision/link_4.stl; visual mesh filename=package://abb_irb4600_40_255/meshes/visual/link_4.stl
- added link r1_link_5, mass 10.00000; collision mesh filename=package://abb_irb4600_40_255/meshes/collision/link_5.stl; visual mesh filename=package://abb_irb4600_40_255/meshes/visual/link_5.stl
- added link r1_link_6, mass 5.00000; collision mesh filename=package://abb_irb4600_40_255/meshes/collision/link_6.stl; visual mesh filename=package://abb_irb4600_40_255/meshes/visual/link_6.stl
- added link r1_tcp
- added link r1_tool0
- added link r2_axis, mass 120; collision mesh filename=package://princeton_cell/meshes/collision/axis.stl; visual mesh filename=package://princeton_cell/meshes/visual/axis.stl
- added link r2_base
- added link r2_base_link, mass 120.00000; collision mesh filename=package://abb_irb4600_40_255/meshes/collision/base_link.stl; visual mesh filename=package://abb_irb4600_40_255/meshes/visual/base_link.stl
- added link r2_cart, mass 120.00000; collision mesh filename=package://princeton_cell/meshes/collision/cart.stl; visual mesh filename=package://princeton_cell/meshes/visual/cart.stl
- added link r2_gripper; collision mesh filename=package://princeton_cell/meshes/collision/gripper.stl; visual mesh filename=package://princeton_cell/meshes/visual/gripper.stl
- added link r2_link_1, mass 120.00000; collision mesh filename=package://abb_irb4600_40_255/meshes/collision/link_1.stl; visual mesh filename=package://abb_irb4600_40_255/meshes/visual/link_1.stl
- added link r2_link_2, mass 120.00000; collision mesh filename=package://abb_irb4600_40_255/meshes/collision/link_2.stl; visual mesh filename=package://abb_irb4600_40_255/meshes/visual/link_2.stl
- added link r2_link_3, mass 120.00000; collision mesh filename=package://abb_irb4600_40_255/meshes/collision/link_3.stl; visual mesh filename=package://abb_irb4600_40_255/meshes/visual/link_3.stl
- added link r2_link_4, mass 40.00000; collision mesh filename=package://abb_irb4600_40_255/meshes/collision/link_4.stl; visual mesh filename=package://abb_irb4600_40_255/meshes/visual/link_4.stl
- added link r2_link_5, mass 10.00000; collision mesh filename=package://abb_irb4600_40_255/meshes/collision/link_5.stl; visual mesh filename=package://abb_irb4600_40_255/meshes/visual/link_5.stl
- added link r2_link_6, mass 5.00000; collision mesh filename=package://abb_irb4600_40_255/meshes/collision/link_6.stl; visual mesh filename=package://abb_irb4600_40_255/meshes/visual/link_6.stl
- added link r2_tcp
- added link r2_tool0
Joints:
- removed joint A_abb_joint
- removed joint A_base_link-base
- removed joint A_cart_joint
- removed joint A_gripper_joint
- removed joint A_joint_1
- removed joint A_joint_2
- removed joint A_joint_3
- removed joint A_joint_4
- removed joint A_joint_5
- removed joint A_joint_6
- removed joint A_joint_6-tool0
- removed joint A_tcp_joint
- removed joint A_world_joint
- removed joint B_abb_joint
- removed joint B_base_link-base
- removed joint B_cart_joint
- removed joint B_gripper_joint
- removed joint B_joint_1
- removed joint B_joint_2
- removed joint B_joint_3
- removed joint B_joint_4
- removed joint B_joint_5
- removed joint B_joint_6
- removed joint B_joint_6-tool0
- removed joint B_tcp_joint
- removed joint B_world_joint
- added joint r1_abb_joint: type fixed, parent r1_cart, child r1_base_link, origin xyz=0 0 0  rpy=0 0 -1.5707963267948966
- added joint r1_base_link-base: type fixed, parent r1_base_link, child r1_base, origin xyz=0 0 0 rpy=0 0 0
- added joint r1_cart_joint: type prismatic, parent r1_axis, child r1_cart, origin xyz=0 0 0 rpy=0 0 0, axis 1 0 0, limit lower=0 upper=4.0 effort=100000 velocity=2.618
- added joint r1_gripper_joint: type fixed, parent r1_tool0, child r1_gripper, origin xyz=0 0 0 rpy=0 0 0
- added joint r1_joint_1: type revolute, parent r1_base_link, child r1_link_1, origin xyz=0 0 0 rpy=0 0 0 , axis 0 0 1, limit lower=-3.14159 upper=3.14159 effort=100000 velocity=2.618
- added joint r1_joint_2: type revolute, parent r1_link_1, child r1_link_2, origin xyz=0.175 0 0.495 rpy=0 -0 0 , axis 0 1 0, limit lower=-1.5708 upper=2.61799 effort=100000 velocity=2.618
- added joint r1_joint_3: type revolute, parent r1_link_2, child r1_link_3, origin xyz=0 0 1.095 rpy=0 -0 0 , axis 0 1 0, limit lower=-3.14159 upper=1.309 effort=100000 velocity=2.618
- added joint r1_joint_4: type revolute, parent r1_link_3, child r1_link_4, origin xyz=0.332 0 0.175 rpy=0 -0 0 , axis 1 0 0, limit lower=-6.98132 upper=6.98132 effort=10000 velocity=6.2832
- added joint r1_joint_5: type revolute, parent r1_link_4, child r1_link_5, origin xyz=0.939 0 0 rpy=0 -0 0 , axis 0 1 0, limit lower=-2.18166 upper=2.0944 effort=100000 velocity=6.2832
- added joint r1_joint_6: type revolute, parent r1_link_5, child r1_link_6, origin xyz=0.135 0 0 rpy=0 1.57076 0 , axis 0 0 1, limit lower=-6.98132 upper=6.98132 effort=100000 velocity=7.854
- added joint r1_joint_6-tool0: type fixed, parent r1_link_6, child r1_tool0, origin xyz=0 0 0 rpy=0 0 0
- added joint r1_tcp_joint: type fixed, parent r1_gripper, child r1_tcp, origin xyz=0 0 0.3 rpy=0 0 0
- added joint r1_world_joint: type fixed, parent world, child r1_axis, origin xyz=0.0 3.45 0.02 rpy=0.0 0.0 0
- added joint r2_abb_joint: type fixed, parent r2_cart, child r2_base_link, origin xyz=0 0 0  rpy=0 0 1.5707963267948966
- added joint r2_base_link-base: type fixed, parent r2_base_link, child r2_base, origin xyz=0 0 0 rpy=0 0 0
- added joint r2_cart_joint: type prismatic, parent r2_axis, child r2_cart, origin xyz=0 0 0 rpy=0 0 0, axis 1 0 0, limit lower=0 upper=4.0 effort=100000 velocity=2.618
- added joint r2_gripper_joint: type fixed, parent r2_tool0, child r2_gripper, origin xyz=0 0 0 rpy=0 0 0
- added joint r2_joint_1: type revolute, parent r2_base_link, child r2_link_1, origin xyz=0 0 0 rpy=0 0 0 , axis 0 0 1, limit lower=-3.14159 upper=3.14159 effort=100000 velocity=2.618
- added joint r2_joint_2: type revolute, parent r2_link_1, child r2_link_2, origin xyz=0.175 0 0.495 rpy=0 -0 0 , axis 0 1 0, limit lower=-1.5708 upper=2.61799 effort=100000 velocity=2.618
- added joint r2_joint_3: type revolute, parent r2_link_2, child r2_link_3, origin xyz=0 0 1.095 rpy=0 -0 0 , axis 0 1 0, limit lower=-3.14159 upper=1.309 effort=100000 velocity=2.618
- added joint r2_joint_4: type revolute, parent r2_link_3, child r2_link_4, origin xyz=0.332 0 0.175 rpy=0 -0 0 , axis 1 0 0, limit lower=-6.98132 upper=6.98132 effort=10000 velocity=6.2832
- added joint r2_joint_5: type revolute, parent r2_link_4, child r2_link_5, origin xyz=0.939 0 0 rpy=0 -0 0 , axis 0 1 0, limit lower=-2.18166 upper=2.0944 effort=100000 velocity=6.2832
- added joint r2_joint_6: type revolute, parent r2_link_5, child r2_link_6, origin xyz=0.135 0 0 rpy=0 1.57076 0 , axis 0 0 1, limit lower=-6.98132 upper=6.98132 effort=100000 velocity=7.854
- added joint r2_joint_6-tool0: type fixed, parent r2_link_6, child r2_tool0, origin xyz=0 0 0 rpy=0 0 0
- added joint r2_tcp_joint: type fixed, parent r2_gripper, child r2_tcp, origin xyz=0 0 0.3 rpy=0 0 0
- added joint r2_world_joint: type fixed, parent world, child r2_axis, origin xyz=0.0 0.0 0.0 rpy=0.0 0.0 0.0

File: setup/catkin/princeton_cell/urdf/princeton_cell_macro.xacro (robot description, xacro)
@@ -4,16 +4,16 @@
     <xacro:include filename="$(find princeton_cell)/urdf/abb_on_axis_macro.xacro"/>
     <link name="world" />
-    <joint name="A_world_joint" type="fixed">
+    <joint name="r2_world_joint" type="fixed">
       <parent link="world" />
-      <child link = "A_axis" />
+      <child link = "r2_axis" />
       <origin xyz="0.0 0.0 0.0" rpy="0.0 0.0 0.0" />
     </joint>
-    <xacro:abb_on_axis prefix="A_"/>
-    <joint name="B_world_joint" type="fixed">
+    <xacro:abb_on_axis prefix="r2_" cart_yaw="${pi/2}"/>
+    <joint name="r1_world_joint" type="fixed">
       <parent link="world" />
-      <child link = "B_axis" />
-      <origin rpy="0.0 0.0 3.14159" xyz="3.70 3.45 0.02"/>
+      <child link = "r1_axis" />
+      <origin rpy="0.0 0.0 0" xyz="0.0 3.45 0.02"/>
     </joint>
-    <xacro:abb_on_axis prefix="B_"/>
+    <xacro:abb_on_axis prefix="r1_" cart_yaw="${-pi/2}"/>
   </xacro:macro>
 </robot>

Commit message: Update gripper's geometry and rotation

File: setup/catkin/princeton_cell/urdf/abb_on_axis.urdf (robot description, URDF)
Before this commit: robot abb_on_axis, 13 links, 12 joints
Joints:
- joint cart_joint: origin xyz=0 0 0 rpy=0 0 0 -> xyz=0 0 0 rpy=0 0 0 
- joint gripper_joint: origin xyz=0 0 0 rpy=0 0 0 -> xyz=0 0 0 rpy=0 0 1.5707963267948966
- joint tcp_joint: origin xyz=0 0 0.3 rpy=0 0 0 -> xyz=0 0 0.352 rpy=0 0 0

File: setup/catkin/princeton_cell/urdf/gripper.xacro (robot description, xacro)
@@ -9,5 +9,5 @@
       <child link="${prefix}gripper"/>
       <!-- The tool is directly attached to the flange. -->
-      <origin rpy="0 0 0" xyz="0 0 0"/>
+      <origin rpy="0 0 ${pi/2}" xyz="0 0 0"/>
     </joint>
     <link name="${prefix}gripper">
@@ -27,5 +27,5 @@
     <!-- TCP frame -->
     <joint name="${prefix}tcp_joint" type="fixed">
-      <origin xyz="0 0 0.3" rpy="0 0 0"/>
+      <origin xyz="0 0 0.352" rpy="0 0 0"/>
       <parent link="${prefix}gripper"/>
       <child link="${prefix}tcp"/>

File: setup/catkin/princeton_cell/urdf/princeton_cell.urdf (robot description, URDF)
Before this commit: robot princeton_cell, 27 links, 26 joints
Joints:
- joint r1_cart_joint: origin xyz=0 0 0 rpy=0 0 0 -> xyz=0 0 0 rpy=0 0 0 
- joint r1_gripper_joint: origin xyz=0 0 0 rpy=0 0 0 -> xyz=0 0 0 rpy=0 0 1.5707963267948966
- joint r1_tcp_joint: origin xyz=0 0 0.3 rpy=0 0 0 -> xyz=0 0 0.352 rpy=0 0 0
- joint r2_cart_joint: origin xyz=0 0 0 rpy=0 0 0 -> xyz=0 0 0 rpy=0 0 0 
- joint r2_gripper_joint: origin xyz=0 0 0 rpy=0 0 0 -> xyz=0 0 0 rpy=0 0 1.5707963267948966
- joint r2_tcp_joint: origin xyz=0 0 0.3 rpy=0 0 0 -> xyz=0 0 0.352 rpy=0 0 0

Commit message: The other way around ;)

File: setup/catkin/princeton_cell/urdf/abb_on_axis.urdf (robot description, URDF)
Before this commit: robot abb_on_axis, 13 links, 12 joints
Joints:
- joint gripper_joint: origin xyz=0 0 0 rpy=0 0 1.5707963267948966 -> xyz=0 0 0 rpy=0 0 -1.5707963267948966

File: setup/catkin/princeton_cell/urdf/gripper.xacro (robot description, xacro)
@@ -9,5 +9,5 @@
       <child link="${prefix}gripper"/>
       <!-- The tool is directly attached to the flange. -->
-      <origin rpy="0 0 ${pi/2}" xyz="0 0 0"/>
+      <origin rpy="0 0 ${-pi/2}" xyz="0 0 0"/>
     </joint>
     <link name="${prefix}gripper">

File: setup/catkin/princeton_cell/urdf/princeton_cell.urdf (robot description, URDF)
Before this commit: robot princeton_cell, 27 links, 26 joints
Joints:
- joint r1_gripper_joint: origin xyz=0 0 0 rpy=0 0 1.5707963267948966 -> xyz=0 0 0 rpy=0 0 -1.5707963267948966
- joint r2_gripper_joint: origin xyz=0 0 0 rpy=0 0 1.5707963267948966 -> xyz=0 0 0 rpy=0 0 -1.5707963267948966

Commit message: Fix gripper mesh rotation

File: setup/catkin/princeton_cell/urdf/abb_on_axis.urdf (robot description, URDF)
Before this commit: robot abb_on_axis, 13 links, 12 joints
Joints:
- joint gripper_joint: origin xyz=0 0 0 rpy=0 0 -1.5707963267948966 -> xyz=0 0 0 rpy=0 0 0

File: setup/catkin/princeton_cell/urdf/gripper.xacro (robot description, xacro)
@@ -9,5 +9,5 @@
       <child link="${prefix}gripper"/>
       <!-- The tool is directly attached to the flange. -->
-      <origin rpy="0 0 ${-pi/2}" xyz="0 0 0"/>
+      <origin rpy="0 0 0" xyz="0 0 0"/>
     </joint>
     <link name="${prefix}gripper">

File: setup/catkin/princeton_cell/urdf/princeton_cell.urdf (robot description, URDF)
Before this commit: robot princeton_cell, 27 links, 26 joints
Joints:
- joint r1_gripper_joint: origin xyz=0 0 0 rpy=0 0 -1.5707963267948966 -> xyz=0 0 0 rpy=0 0 0
- joint r2_gripper_joint: origin xyz=0 0 0 rpy=0 0 -1.5707963267948966 -> xyz=0 0 0 rpy=0 0 0

Commit message: Flip tracks

File: setup/catkin/princeton_cell/urdf/abb_on_axis.urdf (robot description, URDF)
Before this commit: robot abb_on_axis, 13 links, 12 joints
Joints:
- joint abb_joint: origin xyz=0 0 0  rpy=0 0 0 -> xyz=0 0 0  rpy=0 0 1.5707963267948966 

File: setup/catkin/princeton_cell/urdf/abb_on_axis.xacro (robot description, xacro)
@@ -2,4 +2,4 @@
 <robot name="abb_on_axis" xmlns:xacro="http://wiki.ros.org/xacro">
   <xacro:include filename="$(find princeton_cell)/urdf/abb_on_axis_macro.xacro"/>
-  <xacro:abb_on_axis prefix="" cart_yaw="0" />
+  <xacro:abb_on_axis prefix="" />
 </robot>

File: setup/catkin/princeton_cell/urdf/abb_on_axis_macro.xacro (robot description, xacro)
@@ -1,5 +1,5 @@
 <?xml version="1.0"?>
 <robot xmlns:xacro="http://wiki.ros.org/xacro">
-  <xacro:macro name="abb_on_axis" params="prefix cart_yaw">
+  <xacro:macro name="abb_on_axis" params="prefix">
     <xacro:include filename="$(find abb_resources)/urdf/common_materials.xacro"/>
     <xacro:include filename="$(find abb_irb4600_40_255)/urdf/abb_irb4600_40_255_macro.xacro"/>
@@ -10,5 +10,5 @@
       <parent link="${prefix}cart"/>
       <child  link="${prefix}base_link"/>
-      <origin xyz="0 0 0 " rpy="0 0 ${cart_yaw}"/>
+      <origin xyz="0 0 0 " rpy="0 0 ${pi/2} "/>
       <dynamics damping="0.2" friction="0" />
     </joint>

File: setup/catkin/princeton_cell/urdf/princeton_cell.urdf (robot description, URDF)
Before this commit: robot princeton_cell, 27 links, 26 joints
Joints:
- joint r1_abb_joint: origin xyz=0 0 0  rpy=0 0 -1.5707963267948966 -> xyz=0 0 0  rpy=0 0 1.5707963267948966 
- joint r1_world_joint: origin xyz=0.0 3.45 0.02 rpy=0.0 0.0 0 -> xyz=3.70 3.45 0.02 rpy=0.0 0.0 3.14159
- joint r2_abb_joint: origin xyz=0 0 0  rpy=0 0 1.5707963267948966 -> xyz=0 0 0  rpy=0 0 1.5707963267948966 

File: setup/catkin/princeton_cell/urdf/princeton_cell_macro.xacro (robot description, xacro)
@@ -9,11 +9,11 @@
       <origin xyz="0.0 0.0 0.0" rpy="0.0 0.0 0.0" />
     </joint>
-    <xacro:abb_on_axis prefix="r2_" cart_yaw="${pi/2}"/>
+    <xacro:abb_on_axis prefix="r2_" />
     <joint name="r1_world_joint" type="fixed">
       <parent link="world" />
       <child link = "r1_axis" />
-      <origin rpy="0.0 0.0 0" xyz="0.0 3.45 0.02"/>
+      <origin rpy="0.0 0.0 3.14159" xyz="3.70 3.45 0.02"/>
     </joint>
-    <xacro:abb_on_axis prefix="r1_" cart_yaw="${-pi/2}"/>
+    <xacro:abb_on_axis prefix="r1_" />
   </xacro:macro>
 </robot>
