Commit message: Limit tracks to 3.9m

File: setup/catkin/princeton_cell/urdf/abb_on_axis.urdf (robot description, URDF)
Before this commit: robot abb_on_axis, 13 links, 12 joints
Joints:
- joint cart_joint: limit lower=0 upper=4.0 effort=100000 velocity=2.618 -> lower=0 upper=3.9 effort=100000 velocity=2.618

File: setup/catkin/princeton_cell/urdf/linear_axis.xacro (robot description, xacro)
@@ -25,5 +25,5 @@
       <origin xyz="0 0 0" rpy="0 0 0 "/>
       <axis   xyz="1 0 0"/>
-      <limit lower="0" upper="4.0" effort="100000" velocity="2.618" />
+      <limit lower="0" upper="3.9" effort="100000" velocity="2.618" />
       <dynamics damping="0.2" friction="0" />
     </joint>

File: setup/catkin/princeton_cell/urdf/princeton_cell.urdf (robot description, URDF)
Before this commit: robot princeton_cell, 27 links, 26 joints
Joints:
- joint r1_cart_joint: limit lower=0 upper=4.0 effort=100000 velocity=2.618 -> lower=0 upper=3.9 effort=100000 velocity=2.618
- joint r2_cart_joint: limit lower=0 upper=4.0 effort=100000 velocity=2.618 -> lower=0 upper=3.9 effort=100000 velocity=2.618
